File: hbridge.kicad_sch (KiCad schematic)
At the start: 18 parts, among them J1 Conn_01x04_Male, J2 Screw_Terminal_01x03, Q1 2N7000, Q2 2N7000, Q3 2N3904, Q4 2N3906, Q5 2N3904, Q6 2N3906, Q7 STP20NF06, Q8 STP20NF06

Commit message: Improved proto layout, snapped to 100 mil
Parts:
- added R1: 100k, Resistor_THT:R_Axial_DIN0204_L3.6mm_D1.6mm_P2.54mm_Vertical, symbol Device:R_US
- renumbered R1 to R2, R2 to R3, R3 to R4, R4 to R5
Connections:
- net +5V: now also R1.2
- net PWM: now also R1.1

Commit message: Reduce layout to 1x1 inch, cleaned up silkscreen
Connections:
- net +5V: now also J1.2 (Pin_2); no longer J1.1 (Pin_1)
- net ~PWM~: now also J1.1 (Pin_1); no longer J1.2 (Pin_2)
Changed lines of the file:
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@@
     (stroke (width 0) (type default) (color 0 0 0 0))
   )
-  (wire (pts (xy 100.33 107.95) (xy 113.03 107.95))
+  (wire (pts (xy 113.03 105.41) (xy 113.03 124.46))
     (stroke (width 0) (type default) (color 0 0 0 0))
   )
@@
     (stroke (width 0) (type default) (color 0 0 0 0))
   )
+  (wire (pts (xy 105.41 102.87) (xy 105.41 107.95))
+    (stroke (width 0) (type default) (color 0 0 0 0))
+  )
   (wire (pts (xy 142.24 73.66) (xy 144.78 73.66))
     (stroke (width 0) (type default) (color 0 0 0 0))
@@
     (stroke (width 0) (type default) (color 0 0 0 0))
   )
-  (wire (pts (xy 113.03 107.95) (xy 113.03 124.46))
-    (stroke (width 0) (type default) (color 0 0 0 0))
-  )
   (wire (pts (xy 109.22 110.49) (xy 109.22 96.52))
     (stroke (width 0) (type default) (color 0 0 0 0))
   )
+  (wire (pts (xy 100.33 105.41) (xy 113.03 105.41))
+    (stroke (width 0) (type default) (color 0 0 0 0))
+  )
   (wire (pts (xy 134.62 73.66) (xy 130.81 73.66))
     (stroke (width 0) (type default) (color 0 0 0 0))
@@
   )
   (wire (pts (xy 144.78 85.09) (xy 144.78 91.44))
+    (stroke (width 0) (type default) (color 0 0 0 0))
+  )
+  (wire (pts (xy 105.41 107.95) (xy 100.33 107.95))
     (stroke (width 0) (type default) (color 0 0 0 0))
   )
@@
     (pin "2")
   )
-  (symbol (lib_id "power:+5V") (at 100.33 105.41 0) (unit 1)
+  (symbol (lib_id "power:+5V") (at 105.41 102.87 0) (unit 1)
     (in_bom yes) (on_board yes) (fields_autoplaced)
-    (property "Reference" "#PWR01" (id 0) (at 100.33 109.22 0)
-      (effects (font (size 1.27 1.27)) hide)
-    )
-    (property "Value" "+5V" (id 1) (at 100.33 100.33 0))
-    (property "Footprint" "" (id 2) (at 100.33 105.41 0)
-      (effects (font (size 1.27 1.27)) hide)
-    )
-    (property "Datasheet" "" (id 3) (at 100.33 105.41 0)
-      (effects (font (size 1.27 1.27)) hide)
-    )
+    (property "Reference" "#PWR01" (id 0) (at 105.41 106.68 0)
+      (effects (font (size 1.27 1.27)) hide)
+    )
+    (property "Value" "+5V" (id 1) (at 105.41 97.79 0))
+    (property "Footprint" "" (id 2) (at 105.41 102.87 0)
+      (effects (font (size 1.27 1.27)) hide)
+    )
+    (property "Datasheet" "" (id 3) (at 105.41 102.87 0)
+      (effects (font (size 1.27 1.27)) hide)
+    )
