File: logic.kicad_sch (KiCad schematic)
At the start: 3 parts, among them U21 LM78L05_TO92, U22 74HC00

Commit message: Added bypass cap, tied unused inputs to gnd
Parts:
- added C21: (no value), symbol Device:C
- added unit 2 of U22
Connections:
- net +5V: now also C21.1
- net GND: now also C21.2, U22.4, U22.5
- no-connect marks 0 -> 1
